Commit message: created gazebo world

File: description/robot_core.xacro (robot description, xacro)
@@ -42,4 +42,9 @@
         </xacro:inertial_box>
     </link>
+    <gazebo reference="chassis">
+        <material>
+            Gazebo/White
+        </material>
+    </gazebo>
     <!-- Left wheel link-->
     <joint name='left_wheel_joint' type='continuous'>
@@ -66,4 +71,9 @@
         </xacro:inertial_cylinder>
     </link>
+    <gazebo reference="left_wheel">
+        <material>
+            Gazebo/Blue
+        </material>
+    </gazebo>
     <!-- Right wheel link-->
     <joint name='right_wheel_joint' type='continuous'>
@@ -90,4 +100,9 @@
         </xacro:inertial_cylinder>
     </link>
+    <gazebo reference="right_wheel">
+        <material>
+            Gazebo/Blue
+        </material>
+    </gazebo>
     <!-- caster wheel link-->
     <joint name='caster_wheel_joint' type='fixed'>
@@ -113,3 +128,10 @@
         </xacro:inertial_sphere>
     </link>
+    <gazebo reference="caster_wheel">
+        <material>
+            Gazebo/Black
+        </material>
+        <mu1 value="0.001"/>
+        <mu2 value="0.001"/>
+    </gazebo>
 </robot>
